File: driver.sch (KiCad schematic (older format))
At the start: 10 parts

Commit message: Most of sch ready
Parts:
- added R30: 10k, symbol R
- R31: renamed from R?; value 0R5 -> 0R4
- gave numbers to parts that had none: 9
Connections:
- net GND: now also R30.1
- net PWM: now also R30.2
- net +BATT renamed MOTOR_POWER
Other:
- note added: "No load current\nfor GR42x25: 6.5A"
- note added: "TODO: connect\n"
- note added: "TODO: utile ?"
Changed lines of the file:
@@
 EESchema Schematic File Version 2
 LIBS:hexabot
+LIBS:power
 LIBS:hexabot-cache
 EELAYER 25 0
@@
 $Descr A4 11693 8268
 encoding utf-8
-Sheet 2 3
+Sheet 3 3
 Title ""
 Date ""
@@
 $EndDescr
 $Comp
-L L6201PS U?
+L L6201PS U5
 U 1 1 557880D8
 P 5700 3200
-F 0 "U?" H 5400 3850 60  0000 C CNN
+AR Path="/5578B32E/557880D8" Ref="U5"  Part="1"
+AR Path="/5578F5CB/557880D8" Ref="U6"  Part="1"
+F 0 "U5" H 5400 3850 60  0000 C CNN
 F 1 "L6201PS" H 5550 3950 60  0000 C CNN
 F 2 "" H 5300 3750 60  0000 C CNN
@@
 $EndComp
 $Comp
-L GND #PWR?
+L GND #PWR076
 U 1 1 557880DF
 P 6250 3700
-F 0 "#PWR?" H 6250 3450 50  0001 C CNN
+AR Path="/5578B32E/557880DF" Ref="#PWR076"  Part="1"
+AR Path="/5578F5CB/557880DF" Ref="#PWR086"  Part="1"
+F 0 "#PWR076" H 6250 3450 50  0001 C CNN
 F 1 "GND" H 6250 3550 50  0000 C CNN
 F 2 "" H 6250 3700 60  0000 C CNN
@@
 $EndComp
 $Comp
-L GND #PWR?
+L GND #PWR077
 U 1 1 557880E5
 P 6250 2800
-F 0 "#PWR?" H 6250 2550 50  0001 C CNN
+AR Path="/5578B32E/557880E5" Ref="#PWR077"  Part="1"
+AR Path="/5578F5CB/557880E5" Ref="#PWR087"  Part="1"
+F 0 "#PWR077" H 6250 2550 50  0001 C CNN
 F 1 "GND" H 6250 2650 50  0000 C CNN
 F 2 "" H 6250 2800 60  0000 C CNN
@@
 $EndComp
 $Comp
-L GND #PWR?
+L GND #PWR078
 U 1 1 557880EB
 P 5150 2800
-F 0 "#PWR?" H 5150 2550 50  0001 C CNN
+AR Path="/5578B32E/557880EB" Ref="#PWR078"  Part="1"
+AR Path="/5578F5CB/557880EB" Ref="#PWR088"  Part="1"
+F 0 "#PWR078" H 5150 2550 50  0001 C CNN
 F 1 "GND" H 5150 2650 50  0000 C CNN
 F 2 "" H 5150 2800 60  0000 C CNN
@@
 $EndComp
 $Comp
-L GND #PWR?
+L GND #PWR079
 U 1 1 557880F1
 P 5150 3700
-F 0 "#PWR?" H 5150 3450 50  0001 C CNN
+AR Path="/5578B32E/557880F1" Ref="#PWR079"  Part="1"
+AR Path="/5578F5CB/557880F1" Ref="#PWR089"  Part="1"
+F 0 "#PWR079" H 5150 3450 50  0001 C CNN
 F 1 "GND" H 5150 3550 50  0000 C CNN
 F 2 "" H 5150 3700 60  0000 C CNN
@@
 $EndComp
 $Comp
-L +BATT #PWR?
-U 1 1 557880F7
-P 4100 3150
-F 0 "#PWR?" H 4100 3000 50  0001 C CNN
-F 1 "+BATT" H 4100 3290 50  0000 C CNN
-F 2 "" H 4100 3150 60  0000 C CNN
-F 3 "" H 4100 3150 60  0000 C CNN
-	1    4100 3150
-	1    0    0    -1
-$EndComp
-$Comp
-L C C?
+L C C16
 U 1 1 55788105
 P 4100 3400
-F 0 "C?" H 4125 3500 50  0000 L CNN
+AR Path="/5578B32E/55788105" Ref="C16"  Part="1"
+AR Path="/5578F5CB/55788105" Ref="C21"  Part="1"
+F 0 "C16" H 4125 3500 50  0000 L CNN
 F 1 "100n" H 4125 3300 50  0000 L CNN
 F 2 "" H 4138 3250 30  0000 C CNN
@@
 $EndComp
 $Comp
-L GND #PWR?
+L GND #PWR080
 U 1 1 5578810C
 P 4100 3550
-F 0 "#PWR?" H 4100 3300 50  0001 C CNN
+AR Path="/5578B32E/5578810C" Ref="#PWR080"  Part="1"
+AR Path="/5578F5CB/5578810C" Ref="#PWR090"  Part="1"
+F 0 "#PWR080" H 4100 3300 50  0001 C CNN
 F 1 "GND" H 4100 3400 50  0000 C CNN
 F 2 "" H 4100 3550 60  0000 C CNN
@@
 OUT2
 $Comp
-L C C?
+L C C17
 U 1 1 5578811A
 P 4400 3750
-F 0 "C?" H 4425 3850 50  0000 L CNN
+AR Path="/5578B32E/5578811A" Ref="C17"  Part="1"
+AR Path="/5578F5CB/5578811A" Ref="C22"  Part="1"
+F 0 "C17" H 4425 3850 50  0000 L CNN
 F 1 "15n" H 4425 3650 50  0000 L CNN
 F 2 "" H 4438 3600 30  0000 C CNN
@@
 $EndComp
 $Comp
-L C C?
+L C C19
 U 1 1 55788121
 P 7000 3700
-F 0 "C?" H 7025 3800 50  0000 L CNN
+AR Path="/5578B32E/55788121" Ref="C19"  Part="1"
+AR Path="/5578F5CB/55788121" Ref="C24"  Part="1"
+F 0 "C19" H 7025 3800 50  0000 L CNN
 F 1 "15n" H 7025 3600 50  0000 L CNN
 F 2 "" H 7038 3550 30  0000 C CNN
@@
 	1    0    0    -1
 $EndComp
-Text Label 4850 4000 2    60   ~ 0
+Text Label 4800 4000 2    60   ~ 0
 OUT1
-Text Label 6600 4000 0    60   ~ 0
+Text Label 6650 4000 0    60   ~ 0
 OUT2
 Text HLabel 5000 3500 0    60   Input ~ 0
@@
 PWM
 $Comp
-L R R?
+L R R31
 U 1 1 55788757
 P 7000 3050
-F 0 "R?" V 7080 3050 50  0000 C CNN
-F 1 "0R5" V 7000 3050 50  0000 C CNN
+AR Path="/5578B32E/55788757" Ref="R31"  Part="1"
+AR Path="/5578F5CB/55788757" Ref="R34"  Part="1"
+F 0 "R31" V 7080 3050 50  0000 C CNN
+F 1 "0R4" V 7000 3050 50  0000 C CNN
 F 2 "" V 6930 3050 30  0000 C CNN
 F 3 "" H 7000 3050 30  0000 C CNN
@@
 SENSE
 $Comp
-L GND #PWR?
+L GND #PWR081
 U 1 1 557887AF
 P 7150 3050
-F 0 "#PWR?" H 7150 2800 50  0001 C CNN
+AR Path="/5578B32E/557887AF" Ref="#PWR081"  Part="1"
+AR Path="/5578F5CB/557887AF" Ref="#PWR091"  Part="1"
+F 0 "#PWR081" H 7150 2800 50  0001 C CNN
 F 1 "GND" H 7150 2900 50  0000 C CNN
 F 2 "" H 7150 3050 60  0000 C CNN
@@
 OUT1
 $Comp
-L C C?
+L C C18
 U 1 1 55788975
 P 5550 5000
-F 0 "C?" H 5575 5100 50  0000 L CNN
+AR Path="/5578B32E/55788975" Ref="C18"  Part="1"
+AR Path="/5578F5CB/55788975" Ref="C23"  Part="1"
+F 0 "C18" H 5575 5100 50  0000 L CNN
 F 1 "22n" H 5575 4900 50  0000 L CNN
 F 2 "" H 5588 4850 30  0000 C CNN
@@
 $EndComp
 $Comp
-L R R?
+L R R29
 U 1 1 557889B4
 P 5850 5000
-F 0 "R?" V 5930 5000 50  0000 C CNN
+AR Path="/5578B32E/557889B4" Ref="R29"  Part="1"
+AR Path="/5578F5CB/557889B4" Ref="R32"  Part="1"
+F 0 "R29" V 5930 5000 50  0000 C CNN
 F 1 "10R" V 5850 5000 50  0000 C CNN
 F 2 "" V 5780 5000 30  0000 C CNN
@@
 "Snubber network": NC?
 Wire Wire Line
-	4100 3150 4100 3250
-Wire Wire Line
 	4850 3300 5150 3300
 Wire Wire Line
 	4850 3100 5150 3100
 Wire Wire Line
-	4100 3200 5150 3200
+	3850 3200 5150 3200
 Wire Wire Line
 	4400 3600 4400 3400
@@
 	6000 5000 6300 5000
 $Comp
-L D D?
+L D D11
 U 1 1 55788DDE
 P 4400 4200
-F 0 "D?" H 4400 4300 50  0000 C CNN
+AR Path="/5578B32E/55788DDE" Ref="D11"  Part="1"
+AR Path="/5578F5CB/55788DDE" Ref="D13"  Part="1"
+F 0 "D11" H 4400 4300 50  0000 C CNN
 F 1 "D" H 4400 4100 50  0000 C CNN
 F 2 "" H 4400 4200 60  0000 C CNN
@@
 $EndComp
 $Comp
-L D D?
+L D D12
 U 1 1 55788E84
 P 7000 4200
-F 0 "D?" H 7000 4300 50  0000 C CNN
+AR Path="/5578B32E/55788E84" Ref="D12"  Part="1"
+AR Path="/5578F5CB/55788E84" Ref="D14"  Part="1"
+F 0 "D12" H 7000 4300 50  0000 C CNN
 F 1 "D" H 7000 4100 50  0000 C CNN
 F 2 "" H 7000 4200 60  0000 C CNN
@@
 Connection ~ 4400 4000
 $Comp
-L GND #PWR?
+L GND #PWR082
 U 1 1 55788F78
 P 4400 4350
-F 0 "#PWR?" H 4400 4100 50  0001 C CNN
+AR Path="/5578B32E/55788F78" Ref="#PWR082"  Part="1"
+AR Path="/5578F5CB/55788F78" Ref="#PWR092"  Part="1"
+F 0 "#PWR082" H 4400 4100 50  0001 C CNN
 F 1 "GND" H 4400 4200 50  0000 C CNN
 F 2 "" H 4400 4350 60  0000 C CNN
@@
 $EndComp
 $Comp
-L GND #PWR?
+L GND #PWR083
 U 1 1 55788FAE
 P 7000 4350
-F 0 "#PWR?" H 7000 4100 50  0001 C CNN
+AR Path="/5578B32E/55788FAE" Ref="#PWR083"  Part="1"
+AR Path="/5578F5CB/55788FAE" Ref="#PWR093"  Part="1"
+F 0 "#PWR083" H 7000 4100 50  0001 C CNN
 F 1 "GND" H 7000 4200 50  0000 C CNN
 F 2 "" H 7000 4350 60  0000 C CNN
@@
 BOOT2
 $Comp
-L C C?
+L C C20
 U 1 1 55789138
 P 7350 3450
-F 0 "C?" H 7375 3550 50  0000 L CNN
+AR Path="/5578B32E/55789138" Ref="C20"  Part="1"
+AR Path="/5578F5CB/55789138" Ref="C25"  Part="1"
+F 0 "C20" H 7375 3550 50  0000 L CNN
 F 1 "220n" H 7375 3350 50  0000 L CNN
 F 2 "" H 7388 3300 30  0000 C CNN
@@
 $EndComp
 $Comp
-L GND #PWR?
+L GND #PWR084
 U 1 1 55789189
 P 7350 3600
-F 0 "#PWR?" H 7350 3350 50  0001 C CNN
+AR Path="/5578B32E/55789189" Ref="#PWR084"  Part="1"
+AR Path="/5578F5CB/55789189" Ref="#PWR094"  Part="1"
+F 0 "#PWR084" H 7350 3350 50  0001 C CNN
 F 1 "GND" H 7350 3450 50  0000 C CNN
 F 2 "" H 7350 3600 60  0000 C CNN
@@
 	1    0    0    -1
 $EndComp
+Wire Wire Line
+	6350 3100 6350 2900
+Connection ~ 6350 3100
+$Comp
+L R R30
+U 1 1 55798ABA
+P 6600 2900
+AR Path="/5578B32E/55798ABA" Ref="R30"  Part="1"
+AR Path="/5578F5CB/55798ABA" Ref="R33"  Part="1"
+F 0 "R30" V 6680 2900 50  0000 C CNN
+F 1 "10k" V 6600 2900 50  0000 C CNN
+F 2 "" V 6530 2900 30  0000 C CNN
+F 3 "" H 6600 2900 30  0000 C CNN
+	1    6600 2900
+	0    1    1    0
+$EndComp
+Wire Wire Line
+	6350 2900 6450 2900
+$Comp
+L GND #PWR085
+U 1 1 55798BC1
+P 6750 2900
+AR Path="/5578B32E/55798BC1" Ref="#PWR085"  Part="1"
+AR Path="/5578F5CB/55798BC1" Ref="#PWR095"  Part="1"
+F 0 "#PWR085" H 6750 2650 50  0001 C CNN
+F 1 "GND" H 6750 2750 50  0000 C CNN
+F 2 "" H 6750 2900 60  0000 C CNN
+F 3 "" H 6750 2900 60  0000 C CNN
+	1    6750 2900
+	0    -1   -1   0
+$EndComp
+Text Notes 6650 2800 0    60   ~ 0
+TODO: utile ?
+Wire Wire Line
+	4100 3200 4100 3250
+Text HLabel 3850 3200 0    60   Input ~ 0
+MOTOR_POWER
+Text Notes 7500 3000 0    60   ~ 0
+No load current\nfor GR42x25: 6.5A
+Text Notes 5350 4200 0    60   ~ 0
+TODO: connect\n
 $EndSCHEMATC

Commit message: Probably ready for layout
Parts:
- R31: value 0R4 -> 0R1 3W
Connections:
- net GND: now also U5.21 (DIE_ATTACH)
Other:
- note removed: "TODO: connect\n"
- note removed: "TODO: utile ?"
Changed lines of the file:
@@
 $Descr A4 11693 8268
 encoding utf-8
-Sheet 3 3
+Sheet 2 3
 Title ""
 Date ""
@@
 AR Path="/5578B32E/557880D8" Ref="U5"  Part="1"
 AR Path="/5578F5CB/557880D8" Ref="U6"  Part="1"
+AR Path="/557880D8" Ref="U5"  Part="1"
 F 0 "U5" H 5400 3850 60  0000 C CNN
 F 1 "L6201PS" H 5550 3950 60  0000 C CNN
@@
 AR Path="/5578F5CB/55788757" Ref="R34"  Part="1"
 F 0 "R31" V 7080 3050 50  0000 C CNN
-F 1 "0R4" V 7000 3050 50  0000 C CNN
+F 1 "0R1 3W" V 7000 3050 50  0000 C CNN
 F 2 "" V 6930 3050 30  0000 C CNN
 F 3 "" H 7000 3050 30  0000 C CNN
@@
 	0    -1   -1   0
 $EndComp
-Text Notes 6650 2800 0    60   ~ 0
-TODO: utile ?
 Wire Wire Line
 	4100 3200 4100 3250
@@
 Text Notes 7500 3000 0    60   ~ 0
 No load current\nfor GR42x25: 6.5A
-Text Notes 5350 4200 0    60   ~ 0
-TODO: connect\n
+$Comp
+L GND #PWR?
+U 1 1 557A2B97
+P 5700 4000
+AR Path="/5578B32E/557A2B97" Ref="#PWR?"  Part="1"
+AR Path="/5578F5CB/557A2B97" Ref="#PWR?"  Part="1"
+F 0 "#PWR?" H 5700 3750 50  0001 C CNN
+F 1 "GND" H 5700 3850 50  0000 C CNN
+F 2 "" H 5700 4000 60  0000 C CNN
+F 3 "" H 5700 4000 60  0000 C CNN
+	1    5700 4000
+	1    0    0    -1
+$EndComp
 $EndSCHEMATC

Commit message: DRC
Changed lines of the file:
@@
 LIBS:hexabot
 LIBS:power
+LIBS:device
+LIBS:conn
 LIBS:hexabot-cache
 EELAYER 25 0
@@
 AR Path="/5578F5CB/557880D8" Ref="U6"  Part="1"
 AR Path="/557880D8" Ref="U5"  Part="1"
-F 0 "U5" H 5400 3850 60  0000 C CNN
+F 0 "U6" H 5400 3850 60  0000 C CNN
 F 1 "L6201PS" H 5550 3950 60  0000 C CNN
 F 2 "" H 5300 3750 60  0000 C CNN
@@
 $EndComp
 $Comp
-L GND #PWR076
+L GND #PWR79
 U 1 1 557880DF
 P 6250 3700
-AR Path="/5578B32E/557880DF" Ref="#PWR076"  Part="1"
-AR Path="/5578F5CB/557880DF" Ref="#PWR086"  Part="1"
-F 0 "#PWR076" H 6250 3450 50  0001 C CNN
+AR Path="/5578B32E/557880DF" Ref="#PWR79"  Part="1"
+AR Path="/5578F5CB/557880DF" Ref="#PWR90"  Part="1"
+F 0 "#PWR90" H 6250 3450 50  0001 C CNN
 F 1 "GND" H 6250 3550 50  0000 C CNN
 F 2 "" H 6250 3700 60  0000 C CNN
@@
 $EndComp
 $Comp
-L GND #PWR077
+L GND #PWR78
 U 1 1 557880E5
 P 6250 2800
-AR Path="/5578B32E/557880E5" Ref="#PWR077"  Part="1"
-AR Path="/5578F5CB/557880E5" Ref="#PWR087"  Part="1"
-F 0 "#PWR077" H 6250 2550 50  0001 C CNN
+AR Path="/5578B32E/557880E5" Ref="#PWR78"  Part="1"
+AR Path="/5578F5CB/557880E5" Ref="#PWR89"  Part="1"
+F 0 "#PWR89" H 6250 2550 50  0001 C CNN
 F 1 "GND" H 6250 2650 50  0000 C CNN
 F 2 "" H 6250 2800 60  0000 C CNN
@@
 $EndComp
 $Comp
-L GND #PWR078
+L GND #PWR75
 U 1 1 557880EB
 P 5150 2800
-AR Path="/5578B32E/557880EB" Ref="#PWR078"  Part="1"
-AR Path="/5578F5CB/557880EB" Ref="#PWR088"  Part="1"
-F 0 "#PWR078" H 5150 2550 50  0001 C CNN
+AR Path="/5578B32E/557880EB" Ref="#PWR75"  Part="1"
+AR Path="/5578F5CB/557880EB" Ref="#PWR86"  Part="1"
+F 0 "#PWR86" H 5150 2550 50  0001 C CNN
 F 1 "GND" H 5150 2650 50  0000 C CNN
 F 2 "" H 5150 2800 60  0000 C CNN
@@
 $EndComp
 $Comp
-L GND #PWR079
+L GND #PWR76
 U 1 1 557880F1
 P 5150 3700
-AR Path="/5578B32E/557880F1" Ref="#PWR079"  Part="1"
-AR Path="/5578F5CB/557880F1" Ref="#PWR089"  Part="1"
-F 0 "#PWR079" H 5150 3450 50  0001 C CNN
+AR Path="/5578B32E/557880F1" Ref="#PWR76"  Part="1"
+AR Path="/5578F5CB/557880F1" Ref="#PWR87"  Part="1"
+F 0 "#PWR87" H 5150 3450 50  0001 C CNN
 F 1 "GND" H 5150 3550 50  0000 C CNN
 F 2 "" H 5150 3700 60  0000 C CNN
@@
 AR Path="/5578B32E/55788105" Ref="C16"  Part="1"
 AR Path="/5578F5CB/55788105" Ref="C21"  Part="1"
-F 0 "C16" H 4125 3500 50  0000 L CNN
+F 0 "C21" H 4125 3500 50  0000 L CNN
 F 1 "100n" H 4125 3300 50  0000 L CNN
 F 2 "" H 4138 3250 30  0000 C CNN
@@
 $EndComp
 $Comp
-L GND #PWR080
+L GND #PWR73
 U 1 1 5578810C
 P 4100 3550
-AR Path="/5578B32E/5578810C" Ref="#PWR080"  Part="1"
-AR Path="/5578F5CB/5578810C" Ref="#PWR090"  Part="1"
-F 0 "#PWR080" H 4100 3300 50  0001 C CNN
+AR Path="/5578B32E/5578810C" Ref="#PWR73"  Part="1"
+AR Path="/5578F5CB/5578810C" Ref="#PWR84"  Part="1"
+F 0 "#PWR84" H 4100 3300 50  0001 C CNN
 F 1 "GND" H 4100 3400 50  0000 C CNN
 F 2 "" H 4100 3550 60  0000 C CNN
@@
 AR Path="/5578B32E/5578811A" Ref="C17"  Part="1"
 AR Path="/5578F5CB/5578811A" Ref="C22"  Part="1"
-F 0 "C17" H 4425 3850 50  0000 L CNN
+F 0 "C22" H 4425 3850 50  0000 L CNN
 F 1 "15n" H 4425 3650 50  0000 L CNN
 F 2 "" H 4438 3600 30  0000 C CNN
@@
 AR Path="/5578B32E/55788121" Ref="C19"  Part="1"
 AR Path="/5578F5CB/55788121" Ref="C24"  Part="1"
-F 0 "C19" H 7025 3800 50  0000 L CNN
+F 0 "C24" H 7025 3800 50  0000 L CNN
 F 1 "15n" H 7025 3600 50  0000 L CNN
 F 2 "" H 7038 3550 30  0000 C CNN
@@
 AR Path="/5578B32E/55788757" Ref="R31"  Part="1"
 AR Path="/5578F5CB/55788757" Ref="R34"  Part="1"
-F 0 "R31" V 7080 3050 50  0000 C CNN
+F 0 "R34" V 7080 3050 50  0000 C CNN
 F 1 "0R1 3W" V 7000 3050 50  0000 C CNN
 F 2 "" V 6930 3050 30  0000 C CNN
@@
 SENSE
 $Comp
-L GND #PWR081
+L GND #PWR82
 U 1 1 557887AF
 P 7150 3050
-AR Path="/5578B32E/557887AF" Ref="#PWR081"  Part="1"
-AR Path="/5578F5CB/557887AF" Ref="#PWR091"  Part="1"
-F 0 "#PWR081" H 7150 2800 50  0001 C CNN
+AR Path="/5578B32E/557887AF" Ref="#PWR82"  Part="1"
+AR Path="/5578F5CB/557887AF" Ref="#PWR93"  Part="1"
+F 0 "#PWR93" H 7150 2800 50  0001 C CNN
 F 1 "GND" H 7150 2900 50  0000 C CNN
 F 2 "" H 7150 3050 60  0000 C CNN
@@
 AR Path="/5578B32E/55788975" Ref="C18"  Part="1"
 AR Path="/5578F5CB/55788975" Ref="C23"  Part="1"
-F 0 "C18" H 5575 5100 50  0000 L CNN
+F 0 "C23" H 5575 5100 50  0000 L CNN
 F 1 "22n" H 5575 4900 50  0000 L CNN
 F 2 "" H 5588 4850 30  0000 C CNN
@@
 AR Path="/5578B32E/557889B4" Ref="R29"  Part="1"
 AR Path="/5578F5CB/557889B4" Ref="R32"  Part="1"
-F 0 "R29" V 5930 5000 50  0000 C CNN
+F 0 "R32" V 5930 5000 50  0000 C CNN
 F 1 "10R" V 5850 5000 50  0000 C CNN
 F 2 "" V 5780 5000 30  0000 C CNN
@@
 AR Path="/5578B32E/55788DDE" Ref="D11"  Part="1"
 AR Path="/5578F5CB/55788DDE" Ref="D13"  Part="1"
-F 0 "D11" H 4400 4300 50  0000 C CNN
+F 0 "D13" H 4400 4300 50  0000 C CNN
 F 1 "D" H 4400 4100 50  0000 C CNN
 F 2 "" H 4400 4200 60  0000 C CNN
@@
 AR Path="/5578B32E/55788E84" Ref="D12"  Part="1"
 AR Path="/5578F5CB/55788E84" Ref="D14"  Part="1"
-F 0 "D12" H 7000 4300 50  0000 C CNN
+F 0 "D14" H 7000 4300 50  0000 C CNN
 F 1 "D" H 7000 4100 50  0000 C CNN
 F 2 "" H 7000 4200 60  0000 C CNN
@@
 Connection ~ 4400 4000
 $Comp
-L GND #PWR082
+L GND #PWR74
 U 1 1 55788F78
 P 4400 4350
-AR Path="/5578B32E/55788F78" Ref="#PWR082"  Part="1"
-AR Path="/5578F5CB/55788F78" Ref="#PWR092"  Part="1"
-F 0 "#PWR082" H 4400 4100 50  0001 C CNN
+AR Path="/5578B32E/55788F78" Ref="#PWR74"  Part="1"
+AR Path="/5578F5CB/55788F78" Ref="#PWR85"  Part="1"
+F 0 "#PWR85" H 4400 4100 50  0001 C CNN
 F 1 "GND" H 4400 4200 50  0000 C CNN
 F 2 "" H 4400 4350 60  0000 C CNN
@@
 $EndComp
 $Comp
-L GND #PWR083
+L GND #PWR81
 U 1 1 55788FAE
 P 7000 4350
-AR Path="/5578B32E/55788FAE" Ref="#PWR083"  Part="1"
-AR Path="/5578F5CB/55788FAE" Ref="#PWR093"  Part="1"
-F 0 "#PWR083" H 7000 4100 50  0001 C CNN
+AR Path="/5578B32E/55788FAE" Ref="#PWR81"  Part="1"
+AR Path="/5578F5CB/55788FAE" Ref="#PWR92"  Part="1"
+F 0 "#PWR92" H 7000 4100 50  0001 C CNN
 F 1 "GND" H 7000 4200 50  0000 C CNN
 F 2 "" H 7000 4350 60  0000 C CNN
@@
 AR Path="/5578B32E/55789138" Ref="C20"  Part="1"
 AR Path="/5578F5CB/55789138" Ref="C25"  Part="1"
-F 0 "C20" H 7375 3550 50  0000 L CNN
+F 0 "C25" H 7375 3550 50  0000 L CNN
 F 1 "220n" H 7375 3350 50  0000 L CNN
 F 2 "" H 7388 3300 30  0000 C CNN
@@
 $EndComp
 $Comp
-L GND #PWR084
+L GND #PWR83
 U 1 1 55789189
 P 7350 3600
-AR Path="/5578B32E/55789189" Ref="#PWR084"  Part="1"
-AR Path="/5578F5CB/55789189" Ref="#PWR094"  Part="1"
-F 0 "#PWR084" H 7350 3350 50  0001 C CNN
+AR Path="/5578B32E/55789189" Ref="#PWR83"  Part="1"
+AR Path="/5578F5CB/55789189" Ref="#PWR94"  Part="1"
+F 0 "#PWR94" H 7350 3350 50  0001 C CNN
 F 1 "GND" H 7350 3450 50  0000 C CNN
 F 2 "" H 7350 3600 60  0000 C CNN
@@
 AR Path="/5578B32E/55798ABA" Ref="R30"  Part="1"
 AR Path="/5578F5CB/55798ABA" Ref="R33"  Part="1"
-F 0 "R30" V 6680 2900 50  0000 C CNN
+F 0 "R33" V 6680 2900 50  0000 C CNN
 F 1 "10k" V 6600 2900 50  0000 C CNN
 F 2 "" V 6530 2900 30  0000 C CNN
@@
 	6350 2900 6450 2900
 $Comp
-L GND #PWR085
+L GND #PWR80
 U 1 1 55798BC1
 P 6750 2900
-AR Path="/5578B32E/55798BC1" Ref="#PWR085"  Part="1"
-AR Path="/5578F5CB/55798BC1" Ref="#PWR095"  Part="1"
-F 0 "#PWR085" H 6750 2650 50  0001 C CNN
+AR Path="/5578B32E/55798BC1" Ref="#PWR80"  Part="1"
+AR Path="/5578F5CB/55798BC1" Ref="#PWR91"  Part="1"
+F 0 "#PWR91" H 6750 2650 50  0001 C CNN
 F 1 "GND" H 6750 2750 50  0000 C CNN
 F 2 "" H 6750 2900 60  0000 C CNN
@@
 No load current\nfor GR42x25: 6.5A
 $Comp
-L GND #PWR?
+L GND #PWR77
 U 1 1 557A2B97
 P 5700 4000
-AR Path="/5578B32E/557A2B97" Ref="#PWR?"  Part="1"
-AR Path="/5578F5CB/557A2B97" Ref="#PWR?"  Part="1"
-F 0 "#PWR?" H 5700 3750 50  0001 C CNN
+AR Path="/5578B32E/557A2B97" Ref="#PWR77"  Part="1"
+AR Path="/5578F5CB/557A2B97" Ref="#PWR88"  Part="1"
+F 0 "#PWR88" H 5700 3750 50  0001 C CNN
 F 1 "GND" H 5700 3850 50  0000 C CNN
 F 2 "" H 5700 4000 60  0000 C CNN
