File: driver.sch (KiCad schematic (older format))
At the start: 11 parts, among them U5 L6201PS

Commit message: Draft layout with files
Parts:
- C16, C17, C18, C19, C20, R29, R30: footprint hexabot:R_0805_HandSoldering -> Resistors_SMD:R_0805
- D11, D12: footprint (none) -> Diodes_SMD:SOD-123
- R31: footprint hexabot:R_1206_HandSoldering -> Resistors_SMD:R_0805
Changed lines of the file:
@@
 EESchema Schematic File Version 2
 LIBS:hexabot
-LIBS:power
-LIBS:device
-LIBS:conn
 LIBS:hexabot-cache
 EELAYER 25 0
@@
 F 0 "C21" H 4125 3500 50  0000 L CNN
 F 1 "100n" H 4125 3300 50  0000 L CNN
-F 2 "hexabot:R_0805_HandSoldering" H 4138 3250 30  0001 C CNN
+F 2 "Resistors_SMD:R_0805" H 4138 3250 30  0001 C CNN
 F 3 "" H 4100 3400 60  0000 C CNN
 	1    4100 3400
@@
 F 0 "C22" H 4425 3850 50  0000 L CNN
 F 1 "15n" H 4425 3650 50  0000 L CNN
-F 2 "hexabot:R_0805_HandSoldering" H 4438 3600 30  0001 C CNN
+F 2 "Resistors_SMD:R_0805" H 4438 3600 30  0001 C CNN
 F 3 "" H 4400 3750 60  0000 C CNN
 	1    4400 3750
@@
 F 0 "C24" H 7025 3800 50  0000 L CNN
 F 1 "15n" H 7025 3600 50  0000 L CNN
-F 2 "hexabot:R_0805_HandSoldering" H 7038 3550 30  0001 C CNN
+F 2 "Resistors_SMD:R_0805" H 7038 3550 30  0001 C CNN
 F 3 "" H 7000 3700 60  0000 C CNN
 	1    7000 3700
@@
 F 0 "R34" V 7080 3050 50  0000 C CNN
 F 1 "0R1 3W" V 7000 3050 50  0000 C CNN
-F 2 "hexabot:R_1206_HandSoldering" V 6930 3050 30  0001 C CNN
+F 2 "Resistors_SMD:R_0805" V 6930 3050 30  0001 C CNN
 F 3 "" H 7000 3050 30  0000 C CNN
 	1    7000 3050
@@
 F 0 "C23" H 5575 5100 50  0000 L CNN
 F 1 "22n" H 5575 4900 50  0000 L CNN
-F 2 "hexabot:R_0805_HandSoldering" H 5588 4850 30  0001 C CNN
+F 2 "Resistors_SMD:R_0805" H 5588 4850 30  0001 C CNN
 F 3 "" H 5550 5000 60  0000 C CNN
 	1    5550 5000
@@
 F 0 "R32" V 5930 5000 50  0000 C CNN
 F 1 "10R" V 5850 5000 50  0000 C CNN
-F 2 "hexabot:R_0805_HandSoldering" V 5780 5000 30  0001 C CNN
+F 2 "Resistors_SMD:R_0805" V 5780 5000 30  0001 C CNN
 F 3 "" H 5850 5000 30  0000 C CNN
 	1    5850 5000
@@
 F 0 "D13" H 4400 4300 50  0000 C CNN
 F 1 "D" H 4400 4100 50  0000 C CNN
-F 2 "" H 4400 4200 60  0001 C CNN
+F 2 "Diodes_SMD:SOD-123" H 4400 4200 60  0001 C CNN
 F 3 "" H 4400 4200 60  0000 C CNN
 	1    4400 4200
@@
 F 0 "D14" H 7000 4300 50  0000 C CNN
 F 1 "D" H 7000 4100 50  0000 C CNN
-F 2 "" H 7000 4200 60  0001 C CNN
+F 2 "Diodes_SMD:SOD-123" H 7000 4200 60  0001 C CNN
 F 3 "" H 7000 4200 60  0000 C CNN
 	1    7000 4200
@@
 F 0 "C25" H 7375 3550 50  0000 L CNN
 F 1 "220n" H 7375 3350 50  0000 L CNN
-F 2 "hexabot:R_0805_HandSoldering" H 7388 3300 30  0001 C CNN
+F 2 "Resistors_SMD:R_0805" H 7388 3300 30  0001 C CNN
 F 3 "" H 7350 3450 60  0000 C CNN
 	1    7350 3450
@@
 F 0 "R33" V 6680 2900 50  0000 C CNN
 F 1 "10k" V 6600 2900 50  0000 C CNN
-F 2 "hexabot:R_0805_HandSoldering" V 6530 2900 30  0001 C CNN
+F 2 "Resistors_SMD:R_0805" V 6530 2900 30  0001 C CNN
 F 3 "" H 6600 2900 30  0000 C CNN
 	1    6600 2900
