File: driver.sch (KiCad schematic (older format))
At the start: 11 parts, among them U5 L6201PS

Commit message: Rsense footprintf modified. Anular ring adjusted. Ready to order
Parts:
- R31: footprint Resistors_SMD:R_0805 -> Resistors_SMD:R_1206
Changed lines of the file:
@@
 F 0 "R34" V 7080 3050 50  0000 C CNN
 F 1 "0R1 3W" V 7000 3050 50  0000 C CNN
-F 2 "Resistors_SMD:R_0805" V 6930 3050 30  0001 C CNN
+F 2 "Resistors_SMD:R_1206" V 6930 3050 30  0001 C CNN
 F 3 "" H 7000 3050 30  0000 C CNN
 	1    7000 3050
