File: kicad/hexabot.kicad_pcb (KiCad board)
At the start: 2 copper layers, 100 x 100 mm, 125 parts, among them P1 BATTERY, P10 BUMP2, P11 USB_B, P12 DEBUG, P13 NC, P14 MOTOR_R, P15 MOTOR_L, P16 UART1_5V, P17 ENC1, P18 ENC2, P19 ENC3, P2 EXT_POWER, P20 ENC4, P21 UART2_FTDI3V3, P22 NC, P23 START, P24 DYNAMIXEL2, P25 NC, P26 NC, P27 NC, P3 SERVO1, P4 SERVO2, P5 DYNAMIXEL1, P6 PICKIT, P7 PANIC BUTTON, P8 NC, P9 BUMP1, Q1 Q_NMOS_GSD, Q2 Q_NMOS_GSD, Q3 Q_NMOS_GSD, Q4 Q_NMOS_GSD, SW1 PUSH1, SW2 PUSH2, U1 PTN78020 +5V, U2 PTN78020 SERVO, U3 MCP1727, U4 DSPIC33EP256MU806, U5 L6201PS, U6 L6201PS, Y1 8M

Commit message: Fix silkscreen ENC3 => ENC4
Other:
- board text added: "ENC4"
Changed lines of the file:
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@@
     (effects (font (size 1.5 1.5) (thickness 0.3)))
   )
-  (gr_text ENC3 (at 135 48.75) (layer F.SilkS)
+  (gr_text ENC4 (at 135 48.75) (layer F.SilkS)
     (effects (font (size 1.5 1.5) (thickness 0.3)))
   )
